Commit message: attempting to use builtin plugins for d435 camera

File: realsense2_description/urdf/d435.gazebo.xacro (robot description, xacro)
@@ -2,24 +2,21 @@
 <!--
 This is the Gazebo URDF model for the Intel RealSense D435 camera
+Newer Gazebo Harmonic / Ionic sensor documentations: https://gazebosim.org/docs/latest/sensors/
 -->
 <robot xmlns:xacro="http://ros.org/wiki/xacro">
-  <xacro:macro name="gazebo_d435" params="camera_name reference_link topics_ns depth_optical_frame color_optical_frame infrared1_optical_frame infrared2_optical_frame publish_pointcloud:=true" >
+  <xacro:macro name="gazebo_d435" params="camera_name
+                                          reference_link
+                                          topics_ns
+                                          depth_optical_frame
+                                          color_optical_frame
+                                          infrared1_optical_frame
+                                          infrared2_optical_frame
+                                          publish_pointcloud:=false" >
     <!-- Load parameters to model's main link-->
     <xacro:property name="deg_to_rad" value="0.01745329251994329577" />
+    <!-- Define URDF -->
+    <!-- Based on rgbd plugin used in https://github.com/Mechazo11/ros2_asus_xtion -->
     <gazebo reference="${reference_link}">
-      <self_collide>0</self_collide>
-      <enable_wind>0</enable_wind>
-      <kinematic>0</kinematic>
-      <gravity>1</gravity>
-      <!--<mu>1</mu>-->
-      <mu2>1</mu2>
-      <fdir1>0 0 0</fdir1>
-      <!--<slip1>0</slip1>
-      <slip2>0</slip2>-->
-      <kp>1e+13</kp>
-      <kd>1</kd>
-      <!--<max_vel>0.01</max_vel>
-      <min_depth>0</min_depth>-->
-      <sensor name="${camera_name}color" type="camera">
+      <sensor type="camera" name="${camera_name}color">
         <camera name="${camera_name}">
           <horizontal_fov>${69.4*deg_to_rad}</horizontal_fov>

File: realsense2_description/urdf/d435.urdf.xacro (robot description, xacro)
@@ -9,5 +9,5 @@
 <robot name="sensor_d435" xmlns:xacro="http://ros.org/wiki/xacro">
   <!--File includes-->
-  <!-- <xacro:include filename="$(find realsense2_description)/urdf/_d435.gazebo.xacro"/> -->
+  <xacro:include filename="$(find realsense2_gz)/urdf/d435.gazebo.xacro"/>
   <xacro:macro name="sensor_d435" params="name topic_ns parent *origin
                                         update_rate:=30.0
@@ -34,7 +34,9 @@
     <xacro:property name="d435_cam_depth_py" value="0.0175"/>
     <xacro:property name="d435_cam_depth_pz" value="${d435_cam_height/2}"/>
+    <!-- Define material properties for rviz and gazebo -->
     <material name="${name}_aluminum">
     <color rgba="0.5 0.5 0.5 1"/>
     </material>
+    <!-- Define joints and links -->
     <!-- camera body, with origin at bottom screw mount -->
     <joint name="${name}_joint" type="fixed">
@@ -53,7 +55,5 @@
       <origin xyz="${d435_cam_mount_from_center_offset} ${-d435_cam_depth_py} 0" rpy="${M_PI/2} 0 ${M_PI/2}"/>
         <geometry>
-          <!-- <box size="${d435_cam_width} ${d435_cam_height} ${d435_cam_depth}"/> -->
           <mesh filename="package://realsense2_description/meshes/d435.dae" />
-          <!--<mesh filename="package://realsense2_description/meshes/d435/d435.dae" />-->
         </geometry>
         <material name="${name}_aluminum"/>
@@ -67,4 +67,5 @@
       <inertial>
         <!-- The following are not reliable values, and should not be used for modeling -->
+        <!-- NOTE for the purposes of simulation, these values is expected not to affect significantly -->
         <mass value="0.564" />
         <origin xyz="0 0 0" />
@@ -124,6 +125,10 @@
     </joint>
     <link name="${name}_color_optical_frame"/>
-    <!-- Realsense Gazebo Plugin -->
-    <xacro:gazebo_d435 camera_name="${name}" reference_link="${name}_link" topics_ns="${topics_ns}" depth_optical_frame="${name}_depth_optical_frame" color_optical_frame="${name}_color_optical_frame" infrared1_optical_frame="${name}_left_ir_optical_frame" infrared2_optical_frame="${name}_right_ir_optical_frame" publish_pointcloud="${publish_pointcloud}"/>
+    <!-- gazebo_d435 now use newer Gazebo Harmonic or later builtin plugins -->
+    <xacro:gazebo_d435 camera_name="${name}" reference_link="${name}_link" topics_ns="${topics_ns}" depth_optical_frame="${name}_depth_optical_frame" color_optical_frame="${name}_color_optical_frame"
+    infrared1_optical_frame="${name}_left_ir_optical_frame"
+    infrared2_optical_frame="${name}_right_ir_optical_frame"
+    publish_pointcloud="${publish_pointcloud}"/>
+    <!-- Import gazebo specific URDF file that uses builtin camera module -->
   </xacro:macro>
 </robot>

Commit message: camera model works in RVIZ need to finish integration with gazebo

File: realsense2_description/urdf/d435.gazebo.xacro (robot description, xacro)
@@ -111,31 +111,4 @@
       </sensor> -->
     </gazebo>
-    <!-- TODO depricated -->
-    <!-- <gazebo>
-      <plugin name="${topics_ns}" filename="librealsense_gazebo_plugin.so">
-        <prefix>${camera_name}</prefix>
-        <depthUpdateRate>30.0</depthUpdateRate>
-        <colorUpdateRate>30.0</colorUpdateRate>
-        <infraredUpdateRate>30.0</infraredUpdateRate>
-        <depthTopicName>depth/image_raw</depthTopicName>
-        <depthCameraInfoTopicName>depth/camera_info</depthCameraInfoTopicName>
-        <colorTopicName>color/image_raw</colorTopicName>
-        <colorCameraInfoTopicName>color/camera_info</colorCameraInfoTopicName>
-        <infrared1TopicName>infra1/image_raw</infrared1TopicName>
-        <infrared1CameraInfoTopicName>infra1/camera_info</infrared1CameraInfoTopicName>
-        <infrared2TopicName>infra2/image_raw</infrared2TopicName>
-        <infrared2CameraInfoTopicName>infra2/camera_info</infrared2CameraInfoTopicName>
-        <colorOpticalframeName>${color_optical_frame}</colorOpticalframeName>
-        <depthOpticalframeName>${depth_optical_frame}</depthOpticalframeName>
-        <infrared1OpticalframeName>${infrared1_optical_frame}</infrared1OpticalframeName>
-        <infrared2OpticalframeName>${infrared2_optical_frame}</infrared2OpticalframeName>
-        <rangeMinDepth>0.2</rangeMinDepth>
-        <rangeMaxDepth>10.0</rangeMaxDepth>
-        <pointCloud>${publish_pointcloud}</pointCloud>
-        <pointCloudTopicName>depth/color/points</pointCloudTopicName>
-        <pointCloudCutoff>0.25</pointCloudCutoff>
-        <pointCloudCutoffMax>9.0</pointCloudCutoffMax>
-      </plugin>
-    </gazebo> -->
   </xacro:macro>
 </robot>

File: realsense2_description/urdf/d435.urdf.xacro (robot description, xacro)
@@ -9,6 +9,8 @@
 <robot name="sensor_d435" xmlns:xacro="http://ros.org/wiki/xacro">
   <!--File includes-->
-  <xacro:include filename="$(find realsense2_gz)/urdf/d435.gazebo.xacro"/>
-  <xacro:macro name="sensor_d435" params="name topic_ns parent *origin
+  <xacro:include filename="$(find realsense2_description)/urdf/d435.gazebo.xacro"/>
+  <xacro:macro name="sensor_d435" params="name
+                                        topics_ns
+                                        parent *origin
                                         update_rate:=30.0
                                         image_height:=480

Commit message: camera populated in gazebo, needs testing

File: realsense2_description/urdf/d435.gazebo.xacro (robot description, xacro)
@@ -8,5 +8,4 @@
   <xacro:macro name="gazebo_d435" params="camera_name
                                           reference_link
-                                          topics_ns
                                           update_rate:=30.0
                                           image_height:=480

File: realsense2_description/urdf/d435.urdf.xacro (robot description, xacro)
@@ -10,11 +10,9 @@
   <!--File includes-->
   <xacro:include filename="$(find realsense2_description)/urdf/d435.gazebo.xacro"/>
-  <xacro:macro name="sensor_d435" params="name
-                                        topics_ns
-                                        parent *origin
-                                        update_rate:=30.0
-                                        image_height:=480
-                                        image_width:=640
-                                        publish_pointcloud:=false">
+  <xacro:macro name="sensor_d435" params="name parent_link *origin
+                                          update_rate:=30.0
+                                          image_height:=480
+                                          image_width:=640
+                                          publish_pointcloud:=false">
     <!-- Define properties -->
     <xacro:property name="M_PI" value="3.1415926535897931" />
@@ -44,5 +42,5 @@
     <joint name="${name}_joint" type="fixed">
       <xacro:insert_block name="origin" />
-      <parent link="${parent}"/>
+      <parent link="${parent_link}"/>
       <child link="${name}_bottom_screw_frame" />
     </joint>
@@ -130,5 +128,4 @@
     <xacro:gazebo_d435 camera_name="${name}"
     reference_link="${name}_link"
-    topics_ns="${topics_ns}"
     image_height="480"
     image_width="640"
